File: schema/timer.kicad_pcb (KiCad board)
At the start: 2 copper layers, 0 parts

Commit message: next step
Parts:
- added DD1: ATTINY2313, DIP-20__300, F.Cu at (166.4, 69.8)
- added GB1: BAT, SIL-2, F.Cu at (124.5, 108.0)
- added HG1: HG_LED_7SEG_2_1, SIL-9, F.Cu at (167.6, 54.6)
- added Kbd1: KEYBOARD, SIL-7, F.Cu at (163.8, 100.3)
- added R1: R, R4, F.Cu at (215.9, 74.9)
- added R2: R, R4, F.Cu at (213.4, 57.1)
- added R3: R, R4, F.Cu at (191.8, 88.9)
- added SA1: SA_1-2_CL, SIL-2, F.Cu at (134.6, 81.3)
- added SP1: SPEAKER, SIL-2, F.Cu at (138.4, 59.7)
- added VT1: VT_NPN_BCE, TO220_VERT, F.Cu at (201.9, 76.2)
- added VT2: VT_NPN_BCE, TO220_VERT, F.Cu at (195.6, 57.1)
- added VT3: TR_NPN_BCE, TO220_VERT, F.Cu at (179.1, 88.9)

Commit message: next step
Parts:
- removed GB1: BAT, SIL-2
- removed HG1: HG_LED_7SEG_2_1, SIL-9
- removed R1, R2, R3: R, R4
- removed SA1: SA_1-2_CL, SIL-2
- removed SP1: SPEAKER, SIL-2
- removed VT1, VT2: VT_NPN_BCE, TO220_VERT
- removed VT3: TR_NPN_BCE, TO220_VERT
- added 1pin small: VAL**, 1pinsmall, F.Cu at (89.5, 115.6)
- added 1pin small: VAL**, 1pinsmall, F.Cu at (104.8, 91.4)
- added 1pin small: VAL**, 1pinsmall, F.Cu at (104.8, 113.0)
- added 1pin small: VAL**, 1pinsmall, F.Cu at (104.8, 110.5)
- added 1pin small: VAL**, 1pinsmall, F.Cu at (109.9, 113.0)
- added 1pin small: VAL**, 1pinsmall, F.Cu at (112.4, 110.5)
- added 1pin small: VAL**, 1pinsmall, F.Cu at (90.8, 95.2)
- added 1pin small: VAL**, 1pinsmall, F.Cu at (95.9, 91.4)
- added 1pin small: VAL**, 1pinsmall, F.Cu at (114.9, 95.2)
- added 1pin small: VAL**, 1pinsmall, F.Cu at (109.9, 90.2)
- added SIL-12: Val**, SIL-12, F.Cu at (86.4, 106.7)
- moved DD1 78.4 mm to (97.2, 106.7), turned to 90 degrees
- moved Kbd1 55.8 mm to (112.4, 121.9), turned to 180 degrees
Routing:
- net (no net): track 0.00 -> 84.0 mm
- net VCC: track 0.00 -> 43.8 mm
- net N-0000025: track 0.00 -> 40.6 mm
- net GND: track 0.00 -> 40.5 mm
- net N-0000024: track 0.00 -> 35.6 mm
- net N-0000023: track 0.00 -> 30.5 mm
- net N-0000026: track 0.00 -> 29.1 mm
- net N-0000020: track 0.00 -> 20.3 mm
- net N-0000021: track 0.00 -> 10.2 mm
- net N-000005: track 0.00 -> 8.04 mm
- net N-0000022: track 0.00 -> 3.81 mm
Other:
- board outline added: 38.1 x 40.6 mm
- board text added: "+"
- board text added: "-"
