File: schema/timer.kicad_pcb (KiCad board)
At the start: 2 copper layers, 38.1 x 40.6 mm, 13 parts

Commit message: next step
Routing:
- net (no net): track 84.0 -> 234.0 mm

Commit message: next step
Parts:
- moved 1pin small 2.54 mm to (109.9, 110.5)
- moved 1pin small 2.54 mm to (112.4, 113.0)
Changed lines of the file:
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@@
 (kicad_pcb (version 3) (host pcbnew "(2013-07-07 BZR 4022)-stable")
   (general
-    (links 1)
+    (links 0)
     (no_connects 0)
     (area 81.888667 83.693 124.613333 125.73127)
@@
   )
   (setup
-    (last_trace_width 0.254)
+    (last_trace_width 0.8)
     (user_trace_width 0.5)
     (user_trace_width 0.8)
@@
   )
   (module 1pinsmall (layer F.Cu)
-    (at 109.855 113.03)
-    (fp_text reference "1pin small" (at 1.016 -2.032) (layer F.SilkS)
-      (effects (font (size 1.5 1.5) (thickness 0.15)))
-    )
-    (fp_text value VAL** (at 0.508 2.54) (layer F.SilkS)
-      (effects (font (size 1.5 1.5) (thickness 0.15)))
-    )
-    (pad 2 thru_hole circle (at 0 0) (size 2 2) (drill 0.5)
-      (layers *.Cu *.Mask F.SilkS)
-    )
-  )
-  (module 1pinsmall (layer F.Cu)
-    (at 112.395 110.49)
+    (at 109.855 110.49)
+    (fp_text reference "1pin small" (at 1.016 -2.032) (layer F.SilkS)
+      (effects (font (size 1.5 1.5) (thickness 0.15)))
+    )
+    (fp_text value VAL** (at 0.508 2.54) (layer F.SilkS)
+      (effects (font (size 1.5 1.5) (thickness 0.15)))
+    )
+    (pad 2 thru_hole circle (at 0 0) (size 2 2) (drill 0.5)
+      (layers *.Cu *.Mask F.SilkS)
+    )
+  )
+  (module 1pinsmall (layer F.Cu)
+    (at 112.395 113.03)
     (fp_text reference "1pin small" (at 1.016 -2.032) (layer F.SilkS)
       (effects (font (size 1.5 1.5) (thickness 0.15)))
@@
   (segment (start 109.855 90.17) (end 104.775 91.44) (width 0.8) (layer B.Cu) (net 0) (status 20))
   (segment (start 86.36 115.57) (end 89.535 115.57) (width 0.8) (layer B.Cu) (net 0))
-  (segment (start 109.855 113.03) (end 109.855 121.92) (width 0.8) (layer B.Cu) (net 0))
-  (segment (start 112.395 110.49) (end 112.395 121.92) (width 0.8) (layer B.Cu) (net 0))
+  (segment (start 109.855 110.49) (end 109.855 121.92) (width 0.8) (layer B.Cu) (net 0) (status 10))
+  (segment (start 112.395 113.03) (end 112.395 121.92) (width 0.8) (layer B.Cu) (net 0) (status 10))
   (segment (start 100.965 110.49) (end 104.775 110.49) (width 0.8) (layer B.Cu) (net 0) (status 10))
   (segment (start 93.345 97.79) (end 86.36 97.79) (width 0.8) (layer B.Cu) (net 0) (status 10))
