File: schema/timer.sch (KiCad schematic (older format))
At the start: 7 parts

Commit message: next step
Parts:
- removed R?: RES, symbol RES
- added Kbd1: KEYBOARD, symbol KEYBOARD
- added R1, R2, R3: R, symbol R
- added VT2: VT_NPN_BCE, symbol VT_NPN_BCE
- added VT3: TR_NPN_BCE, symbol TR_NPN_BCE
- gave numbers to parts that had none: 6
Connections:
- net labels added: POWER_VCC
- wire segments 0 -> 56
Other:
- moved on the sheet: DD1, GB1, HG1, SA1, SP1, VT1

Commit message: next step
Connections:
- net GND: no longer HG1.2 (H)
- no-connect marks 0 -> 2
Changed lines of the file:
@@
 Sheet 1 1
 Title ""
-Date "7 feb 2014"
+Date "11 feb 2014"
 Rev ""
 Comp ""
@@
 	9350 1850 9150 1850
 $Comp
-L POWER_GND #08
-U 1 1 52F4E9A0
-P 5400 3500
-F 0 "#08" V 5350 3450 60  0001 C CNN
-F 1 "POWER_GND" V 5450 3450 60  0001 C CNN
-F 2 "" H 5400 3500 60  0001 C CNN
-F 3 "" H 5400 3500 60  0001 C CNN
-	1    5400 3500
-	1    0    0    -1
-$EndComp
-Wire Wire Line
-	5400 3500 5400 3400
-$Comp
 L PWR_FLAG #FLG09
 U 1 1 52F4E9E4
@@
 Wire Wire Line
 	8300 2700 8150 2700
+NoConn ~ 5400 3400
+NoConn ~ 7300 2400
 $EndSCHEMATC

Commit message: next step
Parts:
- GB1: value BAT -> 3V
- HG1: value HG_LED_7SEG_2_1 -> DA03-11GWA
- R1, R2, R3: value R -> 1к
Other:
- moved on the sheet: GB1, SA1, SP1, VT3
Changed lines of the file:
@@
 Sheet 1 1
 Title ""
-Date "11 feb 2014"
+Date "14 feb 2014"
 Rev ""
 Comp ""
@@
 L SPEAKER SP1
 U 1 1 52F14041
-P 8550 2400
-F 0 "SP1" H 8450 2650 70  0000 C CNN
-F 1 "SPEAKER" H 8450 2150 70  0001 C CNN
-F 2 "" H 8550 2400 60  0001 C CNN
-F 3 "" H 8550 2400 60  0001 C CNN
-	1    8550 2400
+P 8350 2400
+F 0 "SP1" H 8350 2150 70  0000 C CNN
+F 1 "SPEAKER" H 8250 2150 70  0001 C CNN
+F 2 "" H 8350 2400 60  0001 C CNN
+F 3 "" H 8350 2400 60  0001 C CNN
+	1    8350 2400
 	1    0    0    1
 $EndComp
@@
 L POWER_GND #01
 U 1 1 52F13E15
-P 8300 3900
-F 0 "#01" V 8250 3850 60  0001 C CNN
-F 1 "POWER_GND" V 8350 3850 60  0001 C CNN
-F 2 "" H 8300 3900 60  0001 C CNN
-F 3 "" H 8300 3900 60  0001 C CNN
-	1    8300 3900
+P 8100 3900
+F 0 "#01" V 8050 3850 60  0001 C CNN
+F 1 "POWER_GND" V 8150 3850 60  0001 C CNN
+F 2 "" H 8100 3900 60  0001 C CNN
+F 3 "" H 8100 3900 60  0001 C CNN
+	1    8100 3900
 	1    0    0    -1
 $EndComp
@@
 L BAT GB1
 U 1 1 52F13DFB
-P 9150 2750
-F 0 "GB1" H 9175 2625 60  0000 L CNN
-F 1 "BAT" H 9175 2425 60  0000 L CNN
-F 2 "" H 9150 2750 60  0001 C CNN
-F 3 "" H 9150 2750 60  0001 C CNN
-	1    9150 2750
+P 8950 2750
+F 0 "GB1" H 8975 2625 60  0000 L CNN
+F 1 "3V" H 8975 2425 60  0000 L CNN
+F 2 "" H 8950 2750 60  0001 C CNN
+F 3 "" H 8950 2750 60  0001 C CNN
+	1    8950 2750
 	1    0    0    -1
 $EndComp
@@
 L SA_1-2_CL SA1
 U 1 1 52F13A0C
-P 9150 2300
-F 0 "SA1" V 9150 2100 120 0000 C CNN
-F 1 "SA_1-2_CL" H 9150 2200 60  0001 C CNN
-F 2 "" H 9150 2300 60  0001 C CNN
-F 3 "" H 9150 2300 60  0001 C CNN
-	1    9150 2300
+P 8950 2300
+F 0 "SA1" V 8950 2200 59  0000 C CNN
+F 1 "SA_1-2_CL" H 8950 2200 60  0001 C CNN
+F 2 "" H 8950 2300 60  0001 C CNN
+F 3 "" H 8950 2300 60  0001 C CNN
+	1    8950 2300
 	0    -1   -1   0
 $EndComp
@@
 P 5400 2800
 F 0 "HG1" H 5800 3750 60  0000 C CNN
-F 1 "HG_LED_7SEG_2_1" H 5800 2050 60  0000 C CNN
+F 1 "DA03-11GWA" H 5800 2050 60  0000 C CNN
 F 2 "" H 5400 2800 60  0001 C CNN
 F 3 "" H 5400 2800 60  0001 C CNN
@@
 P 3950 3300
 F 0 "R1" V 4030 3300 50  0000 C CNN
-F 1 "R" V 3950 3300 50  0000 C CNN
+F 1 "1к" V 3950 3300 50  0000 C CNN
 F 2 "" H 3950 3300 60  0000 C CNN
 F 3 "" H 3950 3300 60  0000 C CNN
@@
 L TR_NPN_BCE VT3
 U 1 1 52F4AC00
-P 7850 3000
-F 0 "VT3" V 8400 3050 60  0000 R CNN
-F 1 "TR_NPN_BCE" H 8250 2800 60  0001 R CNN
-F 2 "" H 7850 3000 60  0000 C CNN
-F 3 "" H 7850 3000 60  0000 C CNN
-	1    7850 3000
+P 7650 3000
+F 0 "VT3" H 8050 3250 60  0000 R CNN
+F 1 "TR_NPN_BCE" H 8050 2800 60  0001 R CNN
+F 2 "" H 7650 3000 60  0000 C CNN
+F 3 "" H 7650 3000 60  0000 C CNN
+	1    7650 3000
 	1    0    0    -1
 $EndComp
@@
 P 7200 3000
 F 0 "R3" V 7280 3000 50  0000 C CNN
-F 1 "R" V 7200 3000 50  0000 C CNN
+F 1 "1к" V 7200 3000 50  0000 C CNN
 F 2 "" H 7200 3000 60  0000 C CNN
 F 3 "" H 7200 3000 60  0000 C CNN
@@
 P 4250 3250
 F 0 "R2" V 4330 3250 50  0000 C CNN
-F 1 "R" V 4250 3250 50  0000 C CNN
+F 1 "1к" V 4250 3250 50  0000 C CNN
 F 2 "" H 4250 3250 60  0000 C CNN
 F 3 "" H 4250 3250 60  0000 C CNN
@@
 	6800 3000 6950 3000
 Wire Wire Line
-	8300 3300 8300 3900
-Connection ~ 8300 3800
+	8100 3300 8100 3900
+Connection ~ 8100 3800
 Wire Wire Line
 	6800 3600 6800 3400
@@
 	6800 3200 7300 3200
 Wire Wire Line
-	7300 3200 7300 4250
+	7300 3200 7300 4150
 $Comp
 L POWER_VCC #~02
@@
 L POWER_GND #03
 U 1 1 52F4D89D
-P 9150 3350
-F 0 "#03" V 9100 3300 60  0001 C CNN
-F 1 "POWER_GND" V 9200 3300 60  0001 C CNN
-F 2 "" H 9150 3350 60  0001 C CNN
-F 3 "" H 9150 3350 60  0001 C CNN
-	1    9150 3350
+P 8950 3350
+F 0 "#03" V 8900 3300 60  0001 C CNN
+F 1 "POWER_GND" V 9000 3300 60  0001 C CNN
+F 2 "" H 8950 3350 60  0001 C CNN
+F 3 "" H 8950 3350 60  0001 C CNN
+	1    8950 3350
 	1    0    0    -1
 $EndComp
@@
 L POWER_VCC #~04
 U 1 1 52F4D8A9
-P 9150 1900
-F 0 "#~04" V 8950 1650 60  0001 C CNN
-F 1 "POWER_VCC" H 9300 1800 60  0001 C CNN
-F 2 "" H 9150 1900 60  0000 C CNN
-F 3 "" H 9150 1900 60  0000 C CNN
-	1    9150 1900
-	0    -1   -1   0
-$EndComp
-Wire Wire Line
-	9150 1850 9150 2100
-Connection ~ 9150 1950
-Wire Wire Line
-	9150 2750 9150 2500
-Wire Wire Line
-	9150 3200 9150 3350
+P 8950 1900
+F 0 "#~04" V 8750 1650 60  0001 C CNN
+F 1 "POWER_VCC" H 9100 1800 60  0001 C CNN
+F 2 "" H 8950 1900 60  0000 C CNN
+F 3 "" H 8950 1900 60  0000 C CNN
+	1    8950 1900
+	0    -1   -1   0
+$EndComp
+Wire Wire Line
+	8950 1850 8950 2100
+Connection ~ 8950 1950
+Wire Wire Line
+	8950 2750 8950 2500
+Wire Wire Line
+	8950 3200 8950 3350
 Wire Wire Line
 	5800 2000 5400 2000
@@
 	4250 2950 4250 3000
 Wire Wire Line
-	7300 4250 3950 4250
-Wire Wire Line
-	3950 4250 3950 3550
+	7300 4150 3950 4150
+Wire Wire Line
+	3950 4150 3950 3550
 Wire Wire Line
 	4600 2650 4600 2200
@@
 	5800 3600 5650 3600
 Wire Wire Line
-	5650 3600 5650 4550
-Wire Wire Line
-	5650 4550 7800 4550
-Wire Wire Line
-	7800 4550 7800 2000
-Wire Wire Line
-	7800 2000 7400 2000
+	5650 3600 5650 4400
+Wire Wire Line
+	5650 4400 7750 4400
+Wire Wire Line
+	7750 4400 7750 2000
+Wire Wire Line
+	7750 2000 7400 2000
 Wire Wire Line
 	7400 2000 7400 2100
 Wire Wire Line
-	5800 3800 5800 4400
-Wire Wire Line
-	5800 4400 7700 4400
-Wire Wire Line
-	7700 4400 7700 2100
-Wire Wire Line
-	7700 2100 7500 2100
-Wire Wire Line
-	6800 3800 8500 3800
-Wire Wire Line
-	7450 3000 7850 3000
-Wire Wire Line
-	8300 1950 9150 1950
+	5800 3800 5800 4250
+Wire Wire Line
+	5800 4250 7650 4250
+Wire Wire Line
+	7650 4250 7650 2100
+Wire Wire Line
+	7650 2100 7500 2100
+Wire Wire Line
+	8100 1950 8950 1950
 Wire Wire Line
 	3950 2300 3950 3050
-$Comp
-L PWR_FLAG #FLG06
-U 1 1 52F4E909
-P 8500 3650
-F 0 "#FLG06" H 8500 3920 30  0001 C CNN
-F 1 "PWR_FLAG" H 8500 3880 30  0000 C CNN
-F 2 "" H 8500 3650 60  0000 C CNN
-F 3 "" H 8500 3650 60  0000 C CNN
-	1    8500 3650
-	1    0    0    -1
-$EndComp
-Wire Wire Line
-	8500 3800 8500 3650
-$Comp
-L PWR_FLAG #FLG07
-U 1 1 52F4E954
-P 9350 1850
-F 0 "#FLG07" H 9350 2120 30  0001 C CNN
-F 1 "PWR_FLAG" H 9350 2080 30  0000 C CNN
-F 2 "" H 9350 1850 60  0000 C CNN
-F 3 "" H 9350 1850 60  0000 C CNN
-	1    9350 1850
-	1    0    0    -1
-$EndComp
-Wire Wire Line
-	9350 1850 9150 1850
-$Comp
-L PWR_FLAG #FLG09
-U 1 1 52F4E9E4
-P 6900 3600
-F 0 "#FLG09" H 6900 3870 30  0001 C CNN
-F 1 "PWR_FLAG" H 6900 3830 30  0000 C CNN
-F 2 "" H 6900 3600 60  0000 C CNN
-F 3 "" H 6900 3600 60  0000 C CNN
-	1    6900 3600
-	1    0    0    -1
-$EndComp
-Wire Wire Line
-	8300 2500 8300 2700
-Wire Wire Line
-	8300 1950 8300 2300
-$Comp
-L PWR_FLAG #FLG010
-U 1 1 52F4EA6B
-P 8150 2700
-F 0 "#FLG010" H 8150 2970 30  0001 C CNN
-F 1 "PWR_FLAG" H 8150 2930 30  0000 C CNN
-F 2 "" H 8150 2700 60  0000 C CNN
-F 3 "" H 8150 2700 60  0000 C CNN
-	1    8150 2700
-	1    0    0    -1
-$EndComp
-Wire Wire Line
-	8300 2700 8150 2700
+Wire Wire Line
+	8100 2500 8100 2700
+Wire Wire Line
+	8100 1950 8100 2300
 NoConn ~ 5400 3400
 NoConn ~ 7300 2400
+$Comp
+L POWER_GND #?
+U 1 1 52FDA0A6
+P 6800 3850
+F 0 "#?" V 6750 3800 60  0001 C CNN
+F 1 "POWER_GND" V 6850 3800 60  0001 C CNN
+F 2 "" H 6800 3850 60  0001 C CNN
+F 3 "" H 6800 3850 60  0001 C CNN
+	1    6800 3850
+	1    0    0    -1
+$EndComp
+Wire Wire Line
+	6800 3800 6800 3850
+Wire Wire Line
+	7650 3000 7450 3000
 $EndSCHEMATC

Commit message: next step
Parts:
- SP1: value SPEAKER -> 8 Ом
- VT1, VT2: value VT_NPN_BCE -> КТ315
- VT3: value TR_NPN_BCE -> КТ315
Changed lines of the file:
@@
 P 8350 2400
 F 0 "SP1" H 8350 2150 70  0000 C CNN
-F 1 "SPEAKER" H 8250 2150 70  0001 C CNN
+F 1 "8 Ом" H 8350 2700 70  0000 C CNN
 F 2 "" H 8350 2400 60  0001 C CNN
 F 3 "" H 8350 2400 60  0001 C CNN
@@
 P 4250 2100
 F 0 "VT1" V 4450 2150 60  0000 R CNN
-F 1 "VT_NPN_BCE" V 4300 1900 60  0001 R CNN
+F 1 "КТ315" V 4050 2050 60  0000 R CNN
 F 2 "" H 4250 2100 60  0001 C CNN
 F 3 "" H 4250 2100 60  0001 C CNN
@@
 P 7650 3000
 F 0 "VT3" H 8050 3250 60  0000 R CNN
-F 1 "TR_NPN_BCE" H 8050 2800 60  0001 R CNN
+F 1 "КТ315" H 8050 2800 60  0000 R CNN
 F 2 "" H 7650 3000 60  0000 C CNN
 F 3 "" H 7650 3000 60  0000 C CNN
@@
 P 4250 2750
 F 0 "VT2" V 4450 2800 60  0000 R CNN
-F 1 "VT_NPN_BCE" V 4300 2550 60  0001 R CNN
+F 1 "КТ315" V 4050 2700 60  0000 R CNN
 F 2 "" H 4250 2750 60  0001 C CNN
 F 3 "" H 4250 2750 60  0001 C CNN
@@
 P 5800 2000
 F 0 "DD1" H 6300 2150 60  0000 C CNN
-F 1 "ATTINY2313" H 6300 50  60  0000 C CNN
+F 1 "ATTINY2313" H 6300 0   60  0000 C CNN
 F 2 "" H 5800 2000 60  0001 C CNN
 F 3 "" H 5800 2000 60  0001 C CNN
